Commit message: Adding all code after assignment 5

File: catkin_ws/src/my_robot/urdf/my_robot.xacro (robot description, xacro)
@@ -275,4 +275,11 @@
     <child link="camera"/>
   </joint>
+<joint name="camera_optical_joint" type="fixed">
+    <origin xyz="0 0 0" rpy="-1.5707 0 -1.5707"/>
+    <parent link="camera"/>
+    <child link="camera_link_optical"/>
+  </joint>
+  <link name="camera_link_optical">
+  </link>
 	  <joint name="hokuyo_joint" type="fixed">
     <axis xyz="0 1 0" />
